File: Motor Driver.kicad_pcb (KiCad board)
At the start: 2 copper layers, 103.6 x 67.8 mm, 50 parts, among them CON1 AVR-ISP-6, J1 Conn_01x02, J10 Conn_01x04, J11 Conn_01x02, J2 Conn_01x02, J3 Conn_01x04, J4 Conn_01x04, J5 Conn_01x04, J6 Conn_02x02_Odd_Even, J7 Conn_01x02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

Commit message: updated 3D models
Parts:
- added REF**: 3mm drill, 3mm drill, F.Cu at (94.1, 132.4)
- added REF**: 3mm drill, 3mm drill, F.Cu at (189.7, 132.4)
- added REF**: 3mm drill, 3mm drill, F.Cu at (189.7, 72.6)
- added REF**: 3mm drill, 3mm drill, F.Cu at (94.1, 72.6)
- moved J8 4.45 mm to (101.3, 76.2)
Routing:
- net VCC: track 127.5 -> 143.2 mm
- net GND: track 174.6 -> 180.2 mm
Changed lines of the file:
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@@
   (general
     (links 119)
-    (no_connects 7)
+    (no_connects 0)
     (area 90.056499 68.529999 193.788501 136.448001)
     (thickness 1.6)
     (drawings 9)
-    (tracks 334)
+    (tracks 348)
     (zones 0)
-    (modules 50)
+    (modules 54)
     (nets 50)
   )
@@
     (mod_text_size 1 1)
     (mod_text_width 0.15)
-    (pad_size 1.5 1.5)
-    (pad_drill 0.9)
+    (pad_size 4 4)
+    (pad_drill 3)
     (pad_to_mask_clearance 0)
     (aux_axis_origin 0 0)
@@
     (add_net VCC)
   )
+  (module "3mm drill" (layer F.Cu)
+    (at 94.1065 132.398)
+    (fp_text reference REF** (at 0 3.175) (layer F.SilkS)
+      (effects (font (size 1 1) (thickness 0.15)))
+    )
+    (fp_text value "3mm drill" (at 0 -2.54) (layer F.Fab)
+      (effects (font (size 1 1) (thickness 0.15)))
+    )
+    (pad 1 thru_hole circle (at 0 0) (size 4 4) (drill 3) (layers *.Cu *.Mask)
+      (net 2 GND) (zone_connect 2))
+  )
+  (module "3mm drill" (layer F.Cu)
+    (at 189.7385 132.398)
+    (fp_text reference REF** (at 0 3.175) (layer F.SilkS)
+      (effects (font (size 1 1) (thickness 0.15)))
+    )
+    (fp_text value "3mm drill" (at 0 -2.54) (layer F.Fab)
+      (effects (font (size 1 1) (thickness 0.15)))
+    )
+    (pad 1 thru_hole circle (at 0 0) (size 4 4) (drill 3) (layers *.Cu *.Mask)
+      (net 2 GND) (zone_connect 2))
+  )
+  (module "3mm drill" (layer F.Cu)
+    (at 189.7385 72.58)
+    (fp_text reference REF** (at 0 3.175) (layer F.SilkS)
+      (effects (font (size 1 1) (thickness 0.15)))
+    )
+    (fp_text value "3mm drill" (at 0 -2.54) (layer F.Fab)
+      (effects (font (size 1 1) (thickness 0.15)))
+    )
+    (pad 1 thru_hole circle (at 0 0) (size 4 4) (drill 3) (layers *.Cu *.Mask)
+      (net 2 GND) (zone_connect 2))
+  )
+  (module "3mm drill" (layer F.Cu)
+    (at 94.1065 72.58)
+    (fp_text reference REF** (at 0 3.175) (layer F.SilkS)
+      (effects (font (size 1 1) (thickness 0.15)))
+    )
+    (fp_text value "3mm drill" (at 0 -2.54) (layer F.Fab)
+      (effects (font (size 1 1) (thickness 0.15)))
+    )
+    (pad 1 thru_hole circle (at 0 0) (size 4 4) (drill 3) (layers *.Cu *.Mask)
+      (net 2 GND) (zone_connect 2))
+  )
   (module Capacitors_THT:C_Disc_D3.0mm_W2.0mm_P2.50mm (layer F.Cu)
     (at 135.636 103.6555 90)
@@
   )
   (module Connectors_WAGO:WAGO_734_2pin_Straight_RuggedPads (layer F.Cu)
-    (at 96.901 76.17206 90)
+    (at 101.346 76.17206 90)
     (descr "WAGO, Serie 734, Socket, Stiftleiste, 2 polig, 2 pin, rugged Pads, straight, gerade, Date 05Jul2010,")
     (tags "WAGO, Serie 734, Socket, Stiftleiste, 2 polig, 2 pin, rugged Pads, straight, gerade, Date 05Jul2010,")
@@
     (model ${KISYS3DMOD}/TO_SOT_Packages_THT.3dshapes/TO-220-3_Vertical.wrl
       (at (xyz 0.1 0 0))
-      (scale (xyz 0.393701 0.393701 0.393701))
+      (scale (xyz 1 1 1))
       (rotate (xyz 0 0 0))
     )
@@
       (rotate (xyz 0 0 0))
     )
+    (model Housings_DIP.3dshapes/DIP-28_W7.62mm.wrl
+      (at (xyz 0 0 0))
+      (scale (xyz 1 1 1))
+      (rotate (xyz 0 0 0))
+    )
   )
   (module Housings_DIP:DIP-8_W7.62mm_Socket_LongPads (layer F.Cu)
@@
       (rotate (xyz 0 0 0))
     )
+    (model Housings_DIP.3dshapes/DIP-8_W7.62mm.wrl
+      (at (xyz 0 0 0))
+      (scale (xyz 1 1 1))
+      (rotate (xyz 0 0 0))
+    )
   )
   (module Housings_DIP:DIP-8_W7.62mm_Socket_LongPads (layer F.Cu)
@@
       (rotate (xyz 0 0 0))
     )
+    (model Housings_DIP.3dshapes/DIP-8_W7.62mm.wrl
+      (at (xyz 0 0 0))
+      (scale (xyz 1 1 1))
+      (rotate (xyz 0 0 0))
+    )
   )
   (module Crystals:Crystal_HC18-U_Vertical (layer F.Cu)
@@
     (pad 2 thru_hole oval (at 0 2.54 180) (size 1.7 1.7) (drill 1) (layers *.Cu *.Mask)
       (net 47 "Net-(J11-Pad2)"))
-    (model ${KISYS3DMOD}/Pin_Headers.3dshapes/Pin_Header_Straight_1x02_Pitch2.54mm.wrl
+    (model Connectors_JST.3dshapes/JST_XH_B02B-XH-A_02x2.50mm_Straight.wrl
       (at (xyz 0 0 0))
       (scale (xyz 1 1 1))
-      (rotate (xyz 0 0 0))
+      (rotate (xyz 0 0 90))
     )
   )
@@
   (segment (start 132.334 105.0925) (end 134.199 105.0925) (width 0.4064) (layer B.Cu) (net 1))
   (segment (start 134.199 105.0925) (end 135.636 103.6555) (width 0.4064) (layer B.Cu) (net 1))
+  (segment (start 143.129 74.7395) (end 144.058063 74.7395) (width 0.8) (layer B.Cu) (net 2))
+  (segment (start 144.058063 74.7395) (end 144.729 74.068563) (width 0.8) (layer B.Cu) (net 2))
+  (segment (start 132.1435 74.716) (end 133.072563 74.716) (width 0.8) (layer B.Cu) (net 2))
+  (segment (start 133.072563 74.716) (end 133.7435 74.045063) (width 0.8) (layer B.Cu) (net 2))
+  (segment (start 121.285 74.716) (end 122.214063 74.716) (width 0.8) (layer B.Cu) (net 2))
+  (segment (start 122.214063 74.716) (end 122.885 74.045063) (width 0.8) (layer B.Cu) (net 2))
   (segment (start 102.683563 93.142) (end 102.683563 94.071063) (width 0.6096) (layer B.Cu) (net 2))
   (segment (start 102.683563 94.071063) (end 103.3545 94.742) (width 0.6096) (layer B.Cu) (net 2))
@@
   (segment (start 132.334 100.0125) (end 134.493 100.0125) (width 0.4064) (layer B.Cu) (net 2))
   (segment (start 134.493 100.0125) (end 135.636 101.1555) (width 0.4064) (layer B.Cu) (net 2))
+  (segment (start 111.379 77.95006) (end 101.37394 77.95006) (width 0.8) (layer B.Cu) (net 3))
+  (segment (start 101.37394 77.95006) (end 101.346 77.92212) (width 0.8) (layer B.Cu) (net 3))
+  (segment (start 121.285 77.216) (end 120.355937 77.216) (width 0.8) (layer B.Cu) (net 3))
+  (segment (start 120.355937 77.216) (end 119.685 77.886937) (width 0.8) (layer B.Cu) (net 3))
+  (segment (start 132.1435 77.216) (end 131.214437 77.216) (width 0.8) (layer B.Cu) (net 3))
+  (segment (start 131.214437 77.216) (end 130.5435 77.886937) (width 0.8) (layer B.Cu) (net 3))
+  (segment (start 143.129 77.2395) (end 142.199937 77.2395) (width 0.8) (layer B.Cu) (net 3))
+  (segment (start 142.199937 77.2395) (end 141.529 77.910437) (width 0.8) (layer B.Cu) (net 3))
   (segment (start 96.901 77.92212) (end 96.901 81.445183) (width 0.6096) (layer B.Cu) (net 3))
   (segment (start 93.194331 85.151852) (end 93.194331 89.605074) (width 0.6096) (layer B.Cu) (net 3))
